File: kicad/x2/midi_router.kicad_pcb (KiCad board)
At the start: 2 copper layers, 130 x 70 mm, 61 parts, among them J1 USB_B, J2 DIN-5_180degree, J3 DIN-5_180degree, J4 DIN-5_180degree, J5 DIN-5_180degree, J6 Conn_02x03_Odd_Even, SW1 SW_Push, U1 HCPL2730, U2 ATxmega128A1U-AU, U3 USBLC6-2SC6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

Commit message: x2 prototype: fixing MIDI out connection.
Parts:
- moved R8 4.69 mm to (120.5, 86.2)
- moved R9 4.56 mm to (116.0, 86.2)
- moved R10 4.39 mm to (100.1, 86.3)
- moved R11 4.36 mm to (95.7, 86.3)
Connections:
- R10 pad 1: Net-(J5-Pad4) -> Net-(J5-Pad5)
- R11 pad 2: Net-(J5-Pad5) -> Net-(J5-Pad4)
- R8 pad 1: Net-(J4-Pad4) -> Net-(J4-Pad5)
- R9 pad 2: Net-(J4-Pad5) -> Net-(J4-Pad4)
Routing:
- net +5V: track 126.3 -> 133.4 mm, vias 3 -> 4
- net Net-(R8-Pad2): track 21.2 -> 23.3 mm
- net Net-(R10-Pad2): track 24.9 -> 23.3 mm
