File: kicad/x7-rack/main/midi_router_x7_rack.kicad_sch (KiCad schematic)
At the start: 134 parts, among them J1 DIN-5_180degree, J10 DIN-5_180degree, J11 DIN-5_180degree, J12 DIN-5_180degree, J13 DIN-5_180degree, J14 DIN-5_180degree, J15 USB_B, J16 DS1013-06SSiB1-B-0, J17 Conn_01x04_Male, J18 Conn_02x04_Odd_Even, J19 Conn_02x15_Odd_Even, J2 DIN-5_180degree, J20 Conn_01x04_Male, J3 DIN-5_180degree, J4 DIN-5_180degree, J5 DIN-5_180degree, J6 DIN-5_180degree, J7 DIN-5_180degree, J8 DIN-5_180degree, J9 DIN-5_180degree, U1 HCPL-2631, U1.3 74AHC1G125, U1.4 74AHC1G125, U10 ATxmega128A1U-A, U11 LD1117S33TR_SOT223, U12 USBLC6-2SC6, U2 HCPL-2631, U3 HCPL-2631, U4 HCPL-2631, U5 HCPL-2631, U6 74HCT541, U7 74HCT541, U8 74HCT541, U9 74HCT541, Y1 16MHz

Commit message: Fixing main board issues
- box to ground connection
- RX1 connection
Parts:
- removed C12, C2.1, C2.2, C2.3, C2.4, C2.5, C2.6, C2.7, C2.8, C2.9: 0.01u, Capacitor_SMD:C_0805_2012Metric, symbol Device:C_Small
- removed JP4: SolderJumper_3_Bridged12, Jumper:SolderJumper-3_P1.3mm_Bridged12_RoundedPad1.0x1.5mm_NumberLabels, symbol Jumper:SolderJumper_3_Bridged12
- R8: value 220 -> (none); footprint Resistor_SMD:R_0805_2012Metric -> (none)
Connections:
- net UART1 is gone; now on net RX1F: U1.4.4
- net GND: now also H1.1, H2.1, H3.1, H4.1, H5.1, H6.1, H7.1, H8.1, H9.1, J15.5 (Shield)
- net RX1: now also R8.2
- net U9.17: now also J17.3 (Pin_3)
- net RX1F: now reaches R8.1

Commit message: Updating KiCAD
Parts:
- R8: value (none) -> 100; footprint (none) -> Resistor_SMD:R_0805_2012Metric
