File: kicad/x7-rack/main/midi_router_x7_rack.kicad_pcb (KiCad board)
At the start: 2 copper layers, 340 x 70 mm, 136 parts, among them J1 DIN-5_180degree, J10 DIN-5_180degree, J11 DIN-5_180degree, J12 DIN-5_180degree, J13 DIN-5_180degree, J14 DIN-5_180degree, J15 USB_B, J16 DS1013-06SSiB1-B-0, J17 Conn_01x04_Male, J18 Conn_02x04_Odd_Even, J19 Conn_02x15_Odd_Even, J2 DIN-5_180degree, J20 Conn_01x04_Male, J3 DIN-5_180degree, J4 DIN-5_180degree, J5 DIN-5_180degree, J6 DIN-5_180degree, J7 DIN-5_180degree, J8 DIN-5_180degree, J9 DIN-5_180degree, U1 HCPL-2631, U1.3 74AHC1G125, U1.4 74AHC1G125, U10 ATxmega128A1U-A, U11 LD1117S33TR_SOT223, U12 USBLC6-2SC6, U2 HCPL-2631, U3 HCPL-2631, U4 HCPL-2631, U5 HCPL-2631, U6 74HCT541, U7 74HCT541, U8 74HCT541, U9 74HCT541, Y1 16MHz

Commit message: Fixing main board issues
- box to ground connection
- RX1 connection
Parts:
- removed C12, C2.1, C2.2, C2.3, C2.4, C2.5, C2.6, C2.7, C2.8, C2.9: 0.01u, Capacitor_SMD:C_0805_2012Metric
- removed JP4: SolderJumper_3_Bridged12, Jumper:SolderJumper-3_P1.3mm_Bridged12_RoundedPad1.0x1.5mm_NumberLabels
- R8: value 220 -> 100
- moved R8 197.3 mm to (167.9, 156.3)
Connections:
- H1 pad 1: Net-(C2.1-Pad2) -> GND
- H2 pad 1: Net-(C2.2-Pad2) -> GND
- H3 pad 1: Net-(C2.3-Pad2) -> GND
- H4 pad 1: Net-(C2.4-Pad2) -> GND
- H5 pad 1: Net-(C2.5-Pad2) -> GND
- H6 pad 1: Net-(C2.6-Pad2) -> GND
- H7 pad 1: Net-(C2.7-Pad2) -> GND
- H8 pad 1: Net-(C2.8-Pad2) -> GND
- H9 pad 1: Net-(C2.9-Pad2) -> GND
- J15 pad 5: Net-(C12-Pad2) -> GND
- J17 pad 3: Net-(J17-Pad3) -> U9.17
- R8 pad 1: Net-(JP4-Pad2) -> RX1F
- R8 pad 2: Net-(J17-Pad3) -> RX1
- U1.4 pad 4: UART1 -> RX1F
Routing:
- net Net-(C12-Pad2): track 23.1 -> 0.00 mm
- net GND: track 199.0 -> 177.4 mm, vias 77 -> 68
- net RX1: track 231.9 -> 253.2 mm, vias 2 -> 4
- net U9.17: track 94.5 -> 107.2 mm
- net +5V: track 407.1 -> 398.2 mm
- net Net-(C2.3-Pad2): track 8.12 -> 0.00 mm
- net Net-(C2.4-Pad2): track 7.48 -> 0.00 mm
- net Net-(C2.1-Pad2): track 7.10 -> 0.00 mm
- net Net-(C2.2-Pad2): track 7.06 -> 0.00 mm
- net Net-(C2.8-Pad2): track 6.82 -> 0.00 mm
- net Net-(C2.7-Pad2): track 6.65 -> 0.00 mm
- net Net-(C2.5-Pad2): track 6.15 -> 0.00 mm
- net Net-(J17-Pad3): track 6.00 -> 0.00 mm
- net Net-(C2.9-Pad2): track 5.95 -> 0.00 mm
- net Net-(C2.6-Pad2): track 5.45 -> 0.00 mm
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Other:
- board text added: "2023.03.08"
- board text removed: "2022.11.07"

Commit message: Version update
Other:
- board text added: "2023.06.23"
- board text removed: "2023.03.08"
