File: kicad/x7-rack/led/midi_router_x7_led.kicad_pcb (KiCad board)
At the start: 2 copper layers, 246 x 30 mm, 59 parts, among them J19.2 Conn_02x15_Odd_Even, SW19.1 SW_Push_LED

Commit message: Version update
Parts:
- removed C19.1, C19.2, C19.3, C19.4, C19.5, C19.6: 0.01u, Capacitor_SMD:C_0805_2012Metric
Connections:
- H1 pad 1: Net-(C19.1-Pad2) -> GND
- H2 pad 1: Net-(C19.2-Pad2) -> GND
- H3 pad 1: Net-(C19.3-Pad2) -> GND
- H4 pad 1: Net-(C19.4-Pad2) -> GND
- H5 pad 1: Net-(C19.5-Pad2) -> GND
- H6 pad 1: Net-(C19.6-Pad2) -> GND
Routing:
- net GND: track 69.8 -> 58.0 mm, vias 28 -> 22
- net Net-(C19.6-Pad2): track 7.02 -> 0.00 mm
- net Net-(C19.1-Pad2): track 7.02 -> 0.00 mm
- net Net-(C19.5-Pad2): track 6.46 -> 0.00 mm
- net Net-(C19.4-Pad2): track 6.46 -> 0.00 mm
- net Net-(C19.3-Pad2): track 6.05 -> 0.00 mm
- net Net-(C19.2-Pad2): track 6.00 -> 0.00 mm
Other:
- board text added: "2023.06.23"
- board text removed: "2022.11.07"
