File: kicad/x7-rack/led/midi_router_x7_led.kicad_sch (KiCad schematic)
At the start: 57 parts, among them J19.2 Conn_02x15_Odd_Even, SW19.1 SW_Push_LED

Commit message: Version update
Parts:
- removed C19.1, C19.2, C19.3, C19.4, C19.5, C19.6: 0.01u, Capacitor_SMD:C_0805_2012Metric, symbol Device:C_Small
Connections:
- net GND: now also H1.1, H2.1, H3.1, H4.1, H5.1, H6.1
