File: kicad/x4-top/usb_midi_x4_top.kicad_pcb (KiCad board)
At the start: 2 copper layers, 94 x 44.4 mm, 57 parts, among them J1 Conn_02x10_Odd_Even, J2 Conn_02x03_Odd_Even, SW1 SW_Push, U1 HCPL2730, U2 74HCT541, U3 74HCT541, U4 HCPL2730, U5 ATxmega32A4U-AU, Y1 16MHz

Commit message: Minor tweaks.
Parts:
- R1, R2, R3, R4: value 470 -> 220
- U1, U4: value HCPL2730 -> HCPL2631

Commit message: x4-top KiCad upgrade
Other:
- net class Default removed
- net class Power removed
- net class Thick removed
